Commit message: Add files via upload

File: assig_1/urdf/robot.urdf (robot description, URDF)
Before this commit: robot robot_arm, 8 links, 7 joints
Links:
- added link base_leg; visual cylinder length=0.15 radius=0.35
- link head: geometry visual sphere radius=0.24
Joints:
- added joint base_to_leg: type fixed, parent base_link, child base_leg, origin xyz=0 0 -0.4
- joint head_to_l_eye: origin xyz=0.2 0.08 0 -> xyz=0.22 0.08 0
- joint head_to_r_eye: origin xyz=0.2 -0.08 0 -> xyz=0.22 -0.08 0
